File: PCB/CentralBoard/LightController.kicad_pcb (KiCad board)
At the start: 2 copper layers, 55.9 x 81.3 mm, 74 parts, among them P1 CONN_01X03, P10 CONN_01X03, P11 CONN_01X03, P12 CONN_01X03, P13 CONN_01X03, P14 CONN_01X03, P15 CONN_01X03, P16 CONN_01X03, P17 CONN_01X03, P18 CONN_01X03, P2 CONN_01X10, P3 CONN_01X03, P4 CONN_01X10, P5 CONN_01X03, P6 CONN_01X03, P7 CONN_01X03, P8 CONN_01X03, P9 CONN_01X03, SW1 SW_DIP_x06, U1 LM317_3PinPackage, U2 NCP551, U3 PCA9685, U4 BA4510FVM-GTR, U5 BA4510FVM-GTR, U6 BA4510FVM-GTR, U7 BA4510FVM-GTR

Commit message: Changed transimpedance amps to 5V supply. Finished routing CentralBoard
Parts:
- moved P4 22.9 mm to (139.7, 124.5), turned to 180 degrees
- moved R1 20.6 mm to (124.7, 121.9)
- moved R2 19.2 mm to (124.7, 119.1)
- moved R7 19.2 mm to (124.7, 110.7)
- moved R5 18.5 mm to (124.7, 116.3)
- moved R6 18.5 mm to (124.7, 113.5)
Connections:
- C11 pad 1: +3V3 -> +5V
- C12 pad 1: +3V3 -> +5V
- C13 pad 1: +3V3 -> +5V
- C14 pad 1: +3V3 -> +5V
- C15 pad 1: +3V3 -> +5V
- C16 pad 1: +3V3 -> +5V
- C17 pad 1: +3V3 -> +5V
- C18 pad 1: +3V3 -> +5V
- P13 pad 1: Net-(P13-Pad1) -> /lightInterface/LED8
- R14 pad 2: +3V3 -> +5V
- R19 pad 2: +3V3 -> +5V
- R24 pad 2: +3V3 -> +5V
- R9 pad 2: +3V3 -> +5V
- U4 pad 8: +3V3 -> +5V
- U5 pad 8: +3V3 -> +5V
- U6 pad 8: +3V3 -> +5V
- U7 pad 8: +3V3 -> +5V
Routing:
- net GND: track 51.8 -> 356.8 mm, vias 0 -> 12
- net +5V: track 45.7 -> 249.3 mm, vias 0 -> 7
- net +3V3: track 43.2 -> 101.7 mm, vias 0 -> 2
- net /lightInterface/SENSE3: track 2.55 -> 57.2 mm, vias 0 -> 3
- net /lightInterface/SENSE2: track 2.55 -> 47.8 mm, vias 0 -> 3
- net /lightInterface/SENSE1: track 2.55 -> 43.7 mm, vias 0 -> 3
- net /lightInterface/LED9: track 0.00 -> 40.4 mm, vias 0 -> 1
- net /lightInterface/LED1: track 0.00 -> 39.5 mm, vias 0 -> 1
- net /lightInterface/LED2: track 0.00 -> 38.2 mm, vias 0 -> 1
- net /lightInterface/SENSE4: track 2.42 -> 40.6 mm, vias 0 -> 3
- net /lightInterface/LED3: track 0.00 -> 36.7 mm, vias 0 -> 1
- net /lightInterface/LED4: track 0.00 -> 35.5 mm, vias 0 -> 1
- net /lightInterface/LED5: track 0.00 -> 34.2 mm, vias 0 -> 1
- net Net-(R1-Pad1): track 0.00 -> 33.1 mm, vias 0 -> 2
- net /lightInterface/LED8: track 0.00 -> 32.9 mm, vias 0 -> 1
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- added copper zone on B.Cu, net GND
- added copper zone on F.Cu, net GND
Other:
- board text added: "5V"
- board text added: "A0"
- board text added: "A5"
- board text added: "Battery"
- board text added: "Control"
- board text added: "External Supply"
- board text added: "GND"
- board text added: "Lonnie L. Souder II"
- board text added: "Servo Motor"
