File: PCB/CentralBoard/LightController.kicad_pcb (KiCad board)
At the start: 2 copper layers, 55.9 x 81.3 mm, 74 parts, among them P1 CONN_01X03, P10 CONN_01X03, P11 CONN_01X03, P12 CONN_01X03, P13 CONN_01X03, P14 CONN_01X03, P15 CONN_01X03, P16 CONN_01X03, P17 CONN_01X03, P18 CONN_01X03, P2 CONN_01X10, P3 CONN_01X03, P4 CONN_01X10, P5 CONN_01X03, P6 CONN_01X03, P7 CONN_01X03, P8 CONN_01X03, P9 CONN_01X03, SW1 SW_DIP_x06, U1 LM317_3PinPackage, U2 NCP551, U3 PCA9685, U4 BA4510FVM-GTR, U5 BA4510FVM-GTR, U6 BA4510FVM-GTR, U7 BA4510FVM-GTR

Commit message: Fixed transimpedance amp on layout and generated new Gerbers.
Parts:
- added R29: 1.2k, Resistors_SMD:R_0603, F.Cu at (125.2, 148.8)
- added R30: 1.2k, Resistors_SMD:R_0603, F.Cu at (132.1, 148.7)
- added R31: 1.2k, Resistors_SMD:R_0603, F.Cu at (117.9, 148.7)
- added R32: 1.2k, Resistors_SMD:R_0603, F.Cu at (109.2, 146.1)
- R11, R16, R21, R26: value 10k -> 100k
- R13, R18, R23, R28: value 5.1k -> 2.4k
Connections:
- R12 pad 2: Net-(R11-Pad1) -> GND
- R17 pad 2: Net-(R16-Pad1) -> GND
- R22 pad 2: Net-(R21-Pad1) -> GND
- R27 pad 2: Net-(R26-Pad1) -> GND
- U4 pad 5: GND -> Net-(R11-Pad1)
- U5 pad 5: GND -> Net-(R16-Pad1)
- U6 pad 5: GND -> Net-(R21-Pad1)
- U7 pad 5: GND -> Net-(R26-Pad1)
Routing:
- net GND: track 356.8 -> 312.2 mm
- net Net-(R26-Pad1): track 3.96 -> 11.1 mm
- net Net-(R21-Pad1): track 3.86 -> 10.8 mm
- net Net-(R11-Pad1): track 3.96 -> 10.2 mm
- net Net-(R16-Pad1): track 4.22 -> 9.76 mm
- net +5V: track 249.3 -> 247.6 mm
Other:
- board text added: "Rev 2"
