File: PCB/CentralBoard/LightController.sch (KiCad schematic (older format))
At the start: 11 parts

Commit message: Finished LED driver for controller daughter card
Parts:
- added R? (x6): 10k, symbol R
- added SW?: SW_DIP_x06, symbol SW_DIP_x06
Connections:
- net +3V3: now also SW?.1, SW?.2, SW?.3, SW?.4, SW?.5, SW?.6
- net GND: now also U?.25 (EXTCLK), R?.2, R?.2, R?.2, R?.2, R?.2, R?.2
- net lightInterface/SENSE1: now also P?.3 (P3)
- net lightInterface/SENSE2: now also P?.5 (P5)
- net lightInterface/SENSE3: now also P?.6 (P6)
- net lightInterface/SENSE4: now also P?.9 (P9)
- net at P?.8 (P8): now also U?.23 (~OE)
- net at U?.1 (A0): now also R?.1, SW?.12
- net at U?.2 (A1): now also R?.1, SW?.11
- net at U?.24 (A5): now also SW?.7
- net at U?.3 (A2): now also R?.1, SW?.10
- net at U?.4 (A3): now also R?.1, SW?.9
- net at U?.5 (A4): now also R?.1, SW?.8
Other:
- moved on the sheet: C?, P?, U?

Commit message: Finished CentralBoard schematic and added hardware description section to the README
Parts:
- added B+1, B-1: Mounting_Hole_PAD, Mounting_Holes:MountingHole_2.2mm_M2_Pad, symbol Mounting_Hole_PAD
- added C2, C8: 10n, Capacitors_SMD:C_0805, symbol C
- added C4: 1u, Capacitors_SMD:C_0805, symbol C
- added C6: 10u, Capacitors_SMD:C_0805, symbol C
- added P1, P3: CONN_01X03, Pin_Headers:Pin_Header_Straight_1x03_Pitch2.54mm, symbol CONN_01X03
- added R4: 240, Resistors_SMD:R_0805, symbol R
- added R5: 750, Resistors_SMD:R_0805, symbol R
- added U1: LM317_3PinPackage, TO_SOT_Packages_SMD:SOT-223, symbol LM317_3PinPackage
- C1, C10, C3, C5, C7, C9: renamed from C?; footprint (none) -> Capacitors_SMD:C_0805
- P2, P4: renamed from P?; footprint (none) -> Pin_Headers:Pin_Header_Straight_1x10_Pitch2.54mm
- P5: renamed from P?; footprint (none) -> Pin_Headers:Pin_Header_Straight_1x03_Pitch2.54mm
- R1, R2, R3, R6, R7, R8: renamed from R?; value 10k -> 1M; footprint (none) -> Resistors_SMD:R_0805
- SW1: renamed from SW?; footprint (none) -> MyLib:DIP_SW_219-6LPST
- U2: renamed from U?; footprint (none) -> Housings_SSOP:TSOP-5_1.65x3.05mm_Pitch0.95mm
- U3: renamed from U?; footprint (none) -> Housings_SSOP:TSSOP-28_4.4x9.7mm_Pitch0.65mm
Connections:
- net GND: now also B-1.1, C2.2, C4.2, C6.2, C8.2, P3.1 (P1), R5.2
- net at P2.4 (P4): now also P3.3 (P3)
- net +9V: now reaches C1.1, C3.1, U2.1 (Vin), U2.3 (Enable)
- net +9V: now also C2.1, C4.1, P1.2 (P2), U1.3 (VI)
- new net: R4.2, R5.1, U1.1 (ADJ)
- new net: B+1.1, P1.3 (P3)
- new net +5V: C6.1, C8.1, P3.2 (P2), U1.2 (VO)
- no-connect marks 7 -> 8
Other:
- note added: "Optional Battery or Power Supply"
- note added: "Programmable Device Address"
- note added: "Servo Motor Connection"
- moved on the sheet: C1, C10, C3, C5, C7, C9, P2, P4, P5, R1, R2, R3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

Commit message: Created project specific footprint library. Placed all components. Started traces.
Parts:
- C1, C10, C2, C3, C4, C5, C6, C7, C8, C9: footprint Capacitors_SMD:C_0805 -> Capacitors_SMD:C_0603
- R1, R2, R6, R7, R8: footprint Resistors_SMD:R_0805 -> Resistors_SMD:R_0603
- R3: renamed from R4; footprint Resistors_SMD:R_0805 -> Resistors_SMD:R_0603
- R4: renamed from R5; footprint Resistors_SMD:R_0805 -> Resistors_SMD:R_0603
- R5: renamed from R3; footprint Resistors_SMD:R_0805 -> Resistors_SMD:R_0603
- SW1: footprint MyLib:DIP_SW_219-6LPST -> CentralBoardFootprints:DIP_SW_219-6LPST
Connections:
- net +5V: now also R3.1
- net at SW1.7, U3.24 (A5): now also R8.1
Other:
- moved on the sheet: B+1, B-1, C1, C10, C2, C3, C4, C5, C6, C7, C8, C9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
