File: PCB/CentralBoard/lightInterface.sch (KiCad schematic (older format))
At the start: 13 parts

Commit message: Finished LED driver for controller daughter card
Connections:
- wire segments 54 -> 62
Changed lines of the file:
@@
 $Descr A4 11693 8268
 encoding utf-8
-Sheet 2 2
+Sheet 2 6
 Title ""
 Date ""
@@
 	1    0    0    -1
 $EndComp
-Wire Wire Line
-	2650 4050 2600 4050
-Wire Wire Line
-	2600 4050 2600 4200
-Wire Wire Line
-	3200 4050 3200 4200
-Wire Wire Line
-	2600 4200 9150 4200
-Wire Wire Line
-	9150 4200 9150 4050
-Connection ~ 3200 4200
-Wire Wire Line
-	3750 4050 3750 4200
-Connection ~ 3750 4200
-Wire Wire Line
-	4300 4050 4300 4200
-Connection ~ 4300 4200
-Wire Wire Line
-	4800 4050 4800 4200
-Connection ~ 4800 4200
-Wire Wire Line
-	5350 4050 5350 4200
-Connection ~ 5350 4200
-Wire Wire Line
-	5900 4050 5900 4200
-Connection ~ 5900 4200
-Wire Wire Line
-	6450 4050 6450 4200
-Connection ~ 6450 4200
-Wire Wire Line
-	7000 4050 7000 4200
-Connection ~ 7000 4200
-Wire Wire Line
-	7550 4050 7550 4200
-Connection ~ 7550 4200
-Wire Wire Line
-	8100 4050 8100 4200
-Connection ~ 8100 4200
-Wire Wire Line
-	8650 4050 8650 4200
-Connection ~ 8650 4200
 $Comp
 L +5V #PWR?
@@
 	1    0    0    -1
 $EndComp
-Wire Wire Line
-	2450 3700 2450 3950
-Wire Wire Line
-	2450 3950 2650 3950
-Wire Wire Line
-	3200 3950 3100 3950
-Wire Wire Line
-	3100 3950 3100 3700
-Wire Wire Line
-	2450 3700 9050 3700
-Wire Wire Line
-	3650 3700 3650 3950
-Wire Wire Line
-	3650 3950 3750 3950
-Connection ~ 3100 3700
-Wire Wire Line
-	4200 3700 4200 3950
-Wire Wire Line
-	4200 3950 4300 3950
-Connection ~ 3650 3700
-Wire Wire Line
-	4800 3950 4700 3950
-Wire Wire Line
-	4700 3950 4700 3700
-Connection ~ 4200 3700
-Wire Wire Line
-	5350 3950 5250 3950
-Wire Wire Line
-	5250 3950 5250 3700
-Connection ~ 4700 3700
-Wire Wire Line
-	5900 3950 5800 3950
-Wire Wire Line
-	5800 3950 5800 3700
-Connection ~ 5250 3700
-Wire Wire Line
-	6350 3700 6350 3950
-Wire Wire Line
-	6350 3950 6450 3950
-Connection ~ 5800 3700
-Wire Wire Line
-	6900 3700 6900 3950
-Wire Wire Line
-	6900 3950 7000 3950
-Connection ~ 6350 3700
-Wire Wire Line
-	7450 3700 7450 3950
-Wire Wire Line
-	7450 3950 7550 3950
-Connection ~ 6900 3700
-Wire Wire Line
-	8000 3700 8000 3950
-Wire Wire Line
-	8000 3950 8100 3950
-Connection ~ 7450 3700
-Wire Wire Line
-	8550 3700 8550 3950
-Wire Wire Line
-	8550 3950 8650 3950
-Connection ~ 8000 3700
-Wire Wire Line
-	9050 3700 9050 3950
-Wire Wire Line
-	9050 3950 9150 3950
-Connection ~ 8550 3700
 Text HLabel 2650 3600 1    60   Input ~ 0
 LED1
@@
 Text HLabel 7000 3600 1    60   Input ~ 0
 LED9
-Text HLabel 7550 2600 1    60   Input ~ 0
+Text HLabel 6000 2600 0    60   Input ~ 0
 SENSE1
-Text HLabel 8100 2600 1    60   Input ~ 0
+Text HLabel 6000 2050 0    60   Input ~ 0
 SENSE2
-Text HLabel 8650 2600 1    60   Input ~ 0
+Text HLabel 6000 1500 0    60   Input ~ 0
 SENSE3
-Text HLabel 9150 2600 1    60   Input ~ 0
+Text HLabel 6000 1000 0    60   Input ~ 0
 SENSE4
-Wire Wire Line
-	9150 3850 9150 3600
-Wire Wire Line
-	8650 3600 8650 3850
-Wire Wire Line
-	8100 3850 8100 3600
-Wire Wire Line
-	7550 3600 7550 3850
+$Sheet
+S 6300 1450 600  200
+U 5AC9150E
+F0 "transimpedanceAmp3" 60
+F1 "transimpedanceAmp.sch" 60
+F2 "Iin" I R 6900 1500 60
+F3 "Vout" I L 6300 1500 60
+$EndSheet
+$Sheet
+S 6300 950  600  200
+U 5AC931A3
+F0 "transimpedanceAmp4" 60
+F1 "transimpedanceAmp.sch" 60
+F2 "Iin" I R 6900 1000 60
+F3 "Vout" I L 6300 1000 60
+$EndSheet
+$Sheet
+S 6300 2000 600  200
+U 5AC93322
+F0 "transimpedanceAmp2" 60
+F1 "transimpedanceAmp.sch" 60
+F2 "Iin" I R 6900 2050 60
+F3 "Vout" I L 6300 2050 60
+$EndSheet
+$Sheet
+S 6300 2550 600  200
+U 5AC93462
+F0 "transimpedanceAmp1" 60
+F1 "transimpedanceAmp.sch" 60
+F2 "Iin" I R 6900 2600 60
+F3 "Vout" I L 6300 2600 60
+$EndSheet
+Wire Wire Line
+	2650 4050 2600 4050
+Wire Wire Line
+	2600 4050 2600 4200
+Wire Wire Line
+	3200 4050 3200 4200
+Wire Wire Line
+	2600 4200 9150 4200
+Wire Wire Line
+	9150 4200 9150 4050
+Connection ~ 3200 4200
+Wire Wire Line
+	3750 4050 3750 4200
+Connection ~ 3750 4200
+Wire Wire Line
+	4300 4050 4300 4200
+Connection ~ 4300 4200
+Wire Wire Line
+	4800 4050 4800 4200
+Connection ~ 4800 4200
+Wire Wire Line
+	5350 4050 5350 4200
+Connection ~ 5350 4200
+Wire Wire Line
+	5900 4050 5900 4200
+Connection ~ 5900 4200
+Wire Wire Line
+	6450 4050 6450 4200
+Connection ~ 6450 4200
+Wire Wire Line
+	7000 4050 7000 4200
+Connection ~ 7000 4200
+Wire Wire Line
+	7550 4050 7550 4200
+Connection ~ 7550 4200
+Wire Wire Line
+	8100 4050 8100 4200
+Connection ~ 8100 4200
+Wire Wire Line
+	8650 4050 8650 4200
+Connection ~ 8650 4200
+Wire Wire Line
+	2450 3700 2450 3950
+Wire Wire Line
+	2450 3950 2650 3950
+Wire Wire Line
+	3200 3950 3100 3950
+Wire Wire Line
+	3100 3950 3100 3700
+Wire Wire Line
+	2450 3700 9050 3700
+Wire Wire Line
+	3650 3700 3650 3950
+Wire Wire Line
+	3650 3950 3750 3950
+Connection ~ 3100 3700
+Wire Wire Line
+	4200 3700 4200 3950
+Wire Wire Line
+	4200 3950 4300 3950
+Connection ~ 3650 3700
+Wire Wire Line
+	4800 3950 4700 3950
+Wire Wire Line
+	4700 3950 4700 3700
+Connection ~ 4200 3700
+Wire Wire Line
+	5350 3950 5250 3950
+Wire Wire Line
+	5250 3950 5250 3700
+Connection ~ 4700 3700
+Wire Wire Line
+	5900 3950 5800 3950
+Wire Wire Line
+	5800 3950 5800 3700
+Connection ~ 5250 3700
+Wire Wire Line
+	6350 3700 6350 3950
+Wire Wire Line
+	6350 3950 6450 3950
+Connection ~ 5800 3700
+Wire Wire Line
+	6900 3700 6900 3950
+Wire Wire Line
+	6900 3950 7000 3950
+Connection ~ 6350 3700
+Wire Wire Line
+	7450 3700 7450 3950
+Wire Wire Line
+	7450 3950 7550 3950
+Connection ~ 6900 3700
+Wire Wire Line
+	8000 3700 8000 3950
+Wire Wire Line
+	8000 3950 8100 3950
+Connection ~ 7450 3700
+Wire Wire Line
+	8550 3700 8550 3950
+Wire Wire Line
+	8550 3950 8650 3950
+Connection ~ 8000 3700
+Wire Wire Line
+	9050 3700 9050 3950
+Wire Wire Line
+	9050 3950 9150 3950
+Connection ~ 8550 3700
+Wire Wire Line
+	9150 1000 9150 3850
+Wire Wire Line
+	8650 1500 8650 3850
+Wire Wire Line
+	8100 2050 8100 3850
+Wire Wire Line
+	7550 2600 7550 3850
 Wire Wire Line
 	7000 3850 7000 3600
@@
 Wire Wire Line
 	2650 3850 2650 3600
+Wire Wire Line
+	9150 1000 6900 1000
+Wire Wire Line
+	6900 1500 8650 1500
+Wire Wire Line
+	8100 2050 6900 2050
+Wire Wire Line
+	7550 2600 6900 2600
+Wire Wire Line
+	6300 2600 6000 2600
+Wire Wire Line
+	6000 2050 6300 2050
+Wire Wire Line
+	6300 1500 6000 1500
+Wire Wire Line
+	6000 1000 6300 1000
 $EndSCHEMATC

Commit message: Finished CentralBoard schematic and added hardware description section to the README
Parts:
- P10, P11, P12, P13, P14, P15, P16, P17, P18, P6, P7, P8, P9: renamed from P?; footprint (none) -> Pin_Headers:Pin_Header_Straight_1x03_Pitch2.54mm
Changed lines of the file:
@@
 $EndDescr
 $Comp
-L CONN_01X03 P?
+L CONN_01X03 P10
 U 1 1 5AC88470
 P 5000 3950
-F 0 "P?" H 5000 4150 50  0000 C CNN
+F 0 "P10" H 5000 4150 50  0000 C CNN
 F 1 "CONN_01X03" V 5100 3950 50  0000 C CNN
-F 2 "" H 5000 3950 50  0000 C CNN
+F 2 "Pin_Headers:Pin_Header_Straight_1x03_Pitch2.54mm" H 5000 3950 50  0001 C CNN
 F 3 "" H 5000 3950 50  0000 C CNN
 	1    5000 3950
@@
 $EndComp
 $Comp
-L CONN_01X03 P?
+L CONN_01X03 P11
 U 1 1 5AC88477
 P 5550 3950
-F 0 "P?" H 5550 4150 50  0000 C CNN
+F 0 "P11" H 5550 4150 50  0000 C CNN
 F 1 "CONN_01X03" V 5650 3950 50  0000 C CNN
-F 2 "" H 5550 3950 50  0000 C CNN
+F 2 "Pin_Headers:Pin_Header_Straight_1x03_Pitch2.54mm" H 5550 3950 50  0001 C CNN
 F 3 "" H 5550 3950 50  0000 C CNN
 	1    5550 3950
@@
 $EndComp
 $Comp
-L CONN_01X03 P?
+L CONN_01X03 P12
 U 1 1 5AC8847E
 P 6100 3950
-F 0 "P?" H 6100 4150 50  0000 C CNN
+F 0 "P12" H 6100 4150 50  0000 C CNN
 F 1 "CONN_01X03" V 6200 3950 50  0000 C CNN
-F 2 "" H 6100 3950 50  0000 C CNN
+F 2 "Pin_Headers:Pin_Header_Straight_1x03_Pitch2.54mm" H 6100 3950 50  0001 C CNN
 F 3 "" H 6100 3950 50  0000 C CNN
 	1    6100 3950
@@
 $EndComp
 $Comp
-L CONN_01X03 P?
+L CONN_01X03 P13
 U 1 1 5AC88485
 P 6650 3950
-F 0 "P?" H 6650 4150 50  0000 C CNN
+F 0 "P13" H 6650 4150 50  0000 C CNN
 F 1 "CONN_01X03" V 6750 3950 50  0000 C CNN
-F 2 "" H 6650 3950 50  0000 C CNN
+F 2 "Pin_Headers:Pin_Header_Straight_1x03_Pitch2.54mm" H 6650 3950 50  0001 C CNN
 F 3 "" H 6650 3950 50  0000 C CNN
 	1    6650 3950
@@
 $EndComp
 $Comp
-L CONN_01X03 P?
+L CONN_01X03 P6
 U 1 1 5AC8848C
 P 2850 3950
-F 0 "P?" H 2850 4150 50  0000 C CNN
+F 0 "P6" H 2850 4150 50  0000 C CNN
 F 1 "CONN_01X03" V 2950 3950 50  0000 C CNN
-F 2 "" H 2850 3950 50  0000 C CNN
+F 2 "Pin_Headers:Pin_Header_Straight_1x03_Pitch2.54mm" H 2850 3950 50  0001 C CNN
 F 3 "" H 2850 3950 50  0000 C CNN
 	1    2850 3950
@@
 $EndComp
 $Comp
-L CONN_01X03 P?
+L CONN_01X03 P7
 U 1 1 5AC88493
 P 3400 3950
-F 0 "P?" H 3400 4150 50  0000 C CNN
+F 0 "P7" H 3400 4150 50  0000 C CNN
 F 1 "CONN_01X03" V 3500 3950 50  0000 C CNN
-F 2 "" H 3400 3950 50  0000 C CNN
+F 2 "Pin_Headers:Pin_Header_Straight_1x03_Pitch2.54mm" H 3400 3950 50  0001 C CNN
 F 3 "" H 3400 3950 50  0000 C CNN
 	1    3400 3950
@@
 $EndComp
 $Comp
-L CONN_01X03 P?
+L CONN_01X03 P8
 U 1 1 5AC8849A
 P 3950 3950
-F 0 "P?" H 3950 4150 50  0000 C CNN
+F 0 "P8" H 3950 4150 50  0000 C CNN
 F 1 "CONN_01X03" V 4050 3950 50  0000 C CNN
-F 2 "" H 3950 3950 50  0000 C CNN
+F 2 "Pin_Headers:Pin_Header_Straight_1x03_Pitch2.54mm" H 3950 3950 50  0001 C CNN
 F 3 "" H 3950 3950 50  0000 C CNN
 	1    3950 3950
@@
 $EndComp
 $Comp
-L CONN_01X03 P?
+L CONN_01X03 P9
 U 1 1 5AC884A1
 P 4500 3950
-F 0 "P?" H 4500 4150 50  0000 C CNN
+F 0 "P9" H 4500 4150 50  0000 C CNN
 F 1 "CONN_01X03" V 4600 3950 50  0000 C CNN
-F 2 "" H 4500 3950 50  0000 C CNN
+F 2 "Pin_Headers:Pin_Header_Straight_1x03_Pitch2.54mm" H 4500 3950 50  0001 C CNN
 F 3 "" H 4500 3950 50  0000 C CNN
 	1    4500 3950
@@
 $EndComp
 $Comp
-L CONN_01X03 P?
+L CONN_01X03 P18
 U 1 1 5AC884A8
 P 9350 3950
-F 0 "P?" H 9350 4150 50  0000 C CNN
+F 0 "P18" H 9350 4150 50  0000 C CNN
 F 1 "CONN_01X03" V 9450 3950 50  0000 C CNN
-F 2 "" H 9350 3950 50  0000 C CNN
+F 2 "Pin_Headers:Pin_Header_Straight_1x03_Pitch2.54mm" H 9350 3950 50  0001 C CNN
 F 3 "" H 9350 3950 50  0000 C CNN
 	1    9350 3950
@@
 $EndComp
 $Comp
-L CONN_01X03 P?
+L CONN_01X03 P14
 U 1 1 5AC884AF
 P 7200 3950
-F 0 "P?" H 7200 4150 50  0000 C CNN
+F 0 "P14" H 7200 4150 50  0000 C CNN
 F 1 "CONN_01X03" V 7300 3950 50  0000 C CNN
-F 2 "" H 7200 3950 50  0000 C CNN
+F 2 "Pin_Headers:Pin_Header_Straight_1x03_Pitch2.54mm" H 7200 3950 50  0001 C CNN
 F 3 "" H 7200 3950 50  0000 C CNN
 	1    7200 3950
@@
 $EndComp
 $Comp
-L CONN_01X03 P?
+L CONN_01X03 P15
 U 1 1 5AC884B6
 P 7750 3950
-F 0 "P?" H 7750 4150 50  0000 C CNN
+F 0 "P15" H 7750 4150 50  0000 C CNN
 F 1 "CONN_01X03" V 7850 3950 50  0000 C CNN
-F 2 "" H 7750 3950 50  0000 C CNN
+F 2 "Pin_Headers:Pin_Header_Straight_1x03_Pitch2.54mm" H 7750 3950 50  0001 C CNN
 F 3 "" H 7750 3950 50  0000 C CNN
 	1    7750 3950
@@
 $EndComp
 $Comp
-L CONN_01X03 P?
+L CONN_01X03 P16
 U 1 1 5AC884BD
 P 8300 3950
-F 0 "P?" H 8300 4150 50  0000 C CNN
+F 0 "P16" H 8300 4150 50  0000 C CNN
 F 1 "CONN_01X03" V 8400 3950 50  0000 C CNN
-F 2 "" H 8300 3950 50  0000 C CNN
+F 2 "Pin_Headers:Pin_Header_Straight_1x03_Pitch2.54mm" H 8300 3950 50  0001 C CNN
 F 3 "" H 8300 3950 50  0000 C CNN
 	1    8300 3950
@@
 $EndComp
 $Comp
-L CONN_01X03 P?
+L CONN_01X03 P17
 U 1 1 5AC884C4
 P 8850 3950
-F 0 "P?" H 8850 4150 50  0000 C CNN
+F 0 "P17" H 8850 4150 50  0000 C CNN
 F 1 "CONN_01X03" V 8950 3950 50  0000 C CNN
-F 2 "" H 8850 3950 50  0000 C CNN
+F 2 "Pin_Headers:Pin_Header_Straight_1x03_Pitch2.54mm" H 8850 3950 50  0001 C CNN
 F 3 "" H 8850 3950 50  0000 C CNN
 	1    8850 3950
@@
 $EndComp
 $Comp
-L GND #PWR?
+L GND #PWR027
 U 1 1 5AC8854F
 P 2600 4200
-F 0 "#PWR?" H 2600 3950 50  0001 C CNN
+F 0 "#PWR027" H 2600 3950 50  0001 C CNN
 F 1 "GND" H 2600 4050 50  0000 C CNN
 F 2 "" H 2600 4200 50  0001 C CNN
@@
 $EndComp
 $Comp
-L +5V #PWR?
+L +5V #PWR028
 U 1 1 5AC8934C
 P 2450 3700
-F 0 "#PWR?" H 2450 3550 50  0001 C CNN
+F 0 "#PWR028" H 2450 3550 50  0001 C CNN
 F 1 "+5V" H 2450 3840 50  0000 C CNN
 F 2 "" H 2450 3700 50  0001 C CNN

Commit message: Changed transimpedance amps to 5V supply. Finished routing CentralBoard
Connections:
- net LED8: now also P13.1 (P1)
Changed lines of the file:
@@
 Wire Wire Line
 	6000 1000 6300 1000
+Wire Wire Line
+	6450 3600 6450 3850
 $EndSCHEMATC
