File: PCB/CentralBoard/transimpedanceAmp.sch (KiCad schematic (older format))
At the start: 11 parts

Commit message: Finished CentralBoard schematic and added hardware description section to the README
Parts:
- C11, C12, C13, C14: renamed from C?; footprint (none) -> Capacitors_SMD:C_0805
- R10, R11, R12, R13, R9: renamed from R?; footprint (none) -> Resistors_SMD:R_0805
- U4: renamed from U?; footprint (none) -> Housings_SSOP:MSOP-8_3x3mm_Pitch0.65mm
Connections:
- net GND: now also U4.5 (+); no longer U4.3 (+)
- net Vout: now also U4.7; no longer U4.1
- net at R12.1, R13.2: now also U4.6 (-); no longer U4.2 (-)

Commit message: Created project specific footprint library. Placed all components. Started traces.
Parts:
- removed C13: 10u, Capacitors_SMD:C_0805, symbol C
- removed C14: 100n, Capacitors_SMD:C_0805, symbol C
- C11, C12: footprint Capacitors_SMD:C_0805 -> Capacitors_SMD:C_0603
- R10, R11, R12, R13, R9: footprint Resistors_SMD:R_0805 -> Resistors_SMD:R_0603

Commit message: Changed transimpedance amps to 5V supply. Finished routing CentralBoard
Connections:
- net +3V3 renamed +5V
Changed lines of the file:
@@
 AR Path="/5AC88149/5AC93322/5AC91533" Ref="U6"  Part="1"
 AR Path="/5AC88149/5AC93462/5AC91533" Ref="U7"  Part="1"
-F 0 "U6" H 5450 4050 50  0000 L CNN
+F 0 "U7" H 5450 4050 50  0000 L CNN
 F 1 "BA4510FVM-GTR" H 5450 3650 50  0000 L CNN
 F 2 "Housings_SSOP:MSOP-8_3x3mm_Pitch0.65mm" H 5450 3850 50  0001 C CNN
@@
 AR Path="/5AC88149/5AC93322/5AC9170A" Ref="U6"  Part="2"
 AR Path="/5AC88149/5AC93462/5AC9170A" Ref="U7"  Part="2"
-F 0 "U6" H 6750 3950 50  0000 L CNN
+F 0 "U7" H 6750 3950 50  0000 L CNN
 F 1 "BA4510FVM-GTR" H 6750 3550 50  0000 L CNN
 F 2 "Housings_SSOP:MSOP-8_3x3mm_Pitch0.65mm" H 6750 3750 50  0001 C CNN
@@
 $EndComp
 $Comp
-L +3.3V #PWR029
-U 1 1 5AC9179D
-P 5350 3100
-AR Path="/5AC88149/5AC9150E/5AC9179D" Ref="#PWR029"  Part="1"
-AR Path="/5AC88149/5AC931A3/5AC9179D" Ref="#PWR036"  Part="1"
-AR Path="/5AC88149/5AC93322/5AC9179D" Ref="#PWR043"  Part="1"
-AR Path="/5AC88149/5AC93462/5AC9179D" Ref="#PWR050"  Part="1"
-F 0 "#PWR043" H 5350 2950 50  0001 C CNN
-F 1 "+3.3V" H 5350 3240 50  0000 C CNN
-F 2 "" H 5350 3100 50  0001 C CNN
-F 3 "" H 5350 3100 50  0001 C CNN
-	1    5350 3100
-	1    0    0    -1
-$EndComp
-$Comp
-L GND #PWR030
+L GND #PWR029
 U 1 1 5AC91801
 P 5350 4150
-AR Path="/5AC88149/5AC9150E/5AC91801" Ref="#PWR030"  Part="1"
-AR Path="/5AC88149/5AC931A3/5AC91801" Ref="#PWR037"  Part="1"
-AR Path="/5AC88149/5AC93322/5AC91801" Ref="#PWR044"  Part="1"
-AR Path="/5AC88149/5AC93462/5AC91801" Ref="#PWR051"  Part="1"
-F 0 "#PWR044" H 5350 3900 50  0001 C CNN
+AR Path="/5AC88149/5AC9150E/5AC91801" Ref="#PWR029"  Part="1"
+AR Path="/5AC88149/5AC931A3/5AC91801" Ref="#PWR036"  Part="1"
+AR Path="/5AC88149/5AC93322/5AC91801" Ref="#PWR043"  Part="1"
+AR Path="/5AC88149/5AC93462/5AC91801" Ref="#PWR050"  Part="1"
+F 0 "#PWR050" H 5350 3900 50  0001 C CNN
 F 1 "GND" H 5350 4000 50  0000 C CNN
 F 2 "" H 5350 4150 50  0001 C CNN
@@
 $EndComp
 $Comp
-L GND #PWR031
+L GND #PWR030
 U 1 1 5AC91819
 P 6650 4050
-AR Path="/5AC88149/5AC9150E/5AC91819" Ref="#PWR031"  Part="1"
-AR Path="/5AC88149/5AC931A3/5AC91819" Ref="#PWR038"  Part="1"
-AR Path="/5AC88149/5AC93322/5AC91819" Ref="#PWR045"  Part="1"
-AR Path="/5AC88149/5AC93462/5AC91819" Ref="#PWR052"  Part="1"
-F 0 "#PWR045" H 6650 3800 50  0001 C CNN
+AR Path="/5AC88149/5AC9150E/5AC91819" Ref="#PWR030"  Part="1"
+AR Path="/5AC88149/5AC931A3/5AC91819" Ref="#PWR037"  Part="1"
+AR Path="/5AC88149/5AC93322/5AC91819" Ref="#PWR044"  Part="1"
+AR Path="/5AC88149/5AC93462/5AC91819" Ref="#PWR051"  Part="1"
+F 0 "#PWR051" H 6650 3800 50  0001 C CNN
 F 1 "GND" H 6650 3900 50  0000 C CNN
 F 2 "" H 6650 4050 50  0001 C CNN
@@
 AR Path="/5AC88149/5AC93322/5AC91C57" Ref="R20"  Part="1"
 AR Path="/5AC88149/5AC93462/5AC91C57" Ref="R25"  Part="1"
-F 0 "R20" V 3980 3950 50  0000 C CNN
+F 0 "R25" V 3980 3950 50  0000 C CNN
 F 1 "1M" V 3900 3950 50  0000 C CNN
 F 2 "Resistors_SMD:R_0603" V 3830 3950 50  0001 C CNN
@@
 AR Path="/5AC88149/5AC93322/5AC91CDA" Ref="R19"  Part="1"
 AR Path="/5AC88149/5AC93462/5AC91CDA" Ref="R24"  Part="1"
-F 0 "R19" V 3980 3550 50  0000 C CNN
+F 0 "R24" V 3980 3550 50  0000 C CNN
 F 1 "1M" V 3900 3550 50  0000 C CNN
 F 2 "Resistors_SMD:R_0603" V 3830 3550 50  0001 C CNN
@@
 $EndComp
 $Comp
-L +3.3V #PWR032
-U 1 1 5AC91D43
-P 3900 3400
-AR Path="/5AC88149/5AC9150E/5AC91D43" Ref="#PWR032"  Part="1"
-AR Path="/5AC88149/5AC931A3/5AC91D43" Ref="#PWR039"  Part="1"
-AR Path="/5AC88149/5AC93322/5AC91D43" Ref="#PWR046"  Part="1"
-AR Path="/5AC88149/5AC93462/5AC91D43" Ref="#PWR053"  Part="1"
-F 0 "#PWR046" H 3900 3250 50  0001 C CNN
-F 1 "+3.3V" H 3900 3540 50  0000 C CNN
-F 2 "" H 3900 3400 50  0001 C CNN
-F 3 "" H 3900 3400 50  0001 C CNN
-	1    3900 3400
-	-1   0    0    -1
-$EndComp
-$Comp
-L GND #PWR033
+L GND #PWR031
 U 1 1 5AC91D5F
 P 3900 4100
-AR Path="/5AC88149/5AC9150E/5AC91D5F" Ref="#PWR033"  Part="1"
-AR Path="/5AC88149/5AC931A3/5AC91D5F" Ref="#PWR040"  Part="1"
-AR Path="/5AC88149/5AC93322/5AC91D5F" Ref="#PWR047"  Part="1"
-AR Path="/5AC88149/5AC93462/5AC91D5F" Ref="#PWR054"  Part="1"
-F 0 "#PWR047" H 3900 3850 50  0001 C CNN
+AR Path="/5AC88149/5AC9150E/5AC91D5F" Ref="#PWR031"  Part="1"
+AR Path="/5AC88149/5AC931A3/5AC91D5F" Ref="#PWR038"  Part="1"
+AR Path="/5AC88149/5AC93322/5AC91D5F" Ref="#PWR045"  Part="1"
+AR Path="/5AC88149/5AC93462/5AC91D5F" Ref="#PWR052"  Part="1"
+F 0 "#PWR052" H 3900 3850 50  0001 C CNN
 F 1 "GND" H 3900 3950 50  0000 C CNN
 F 2 "" H 3900 4100 50  0001 C CNN
@@
 AR Path="/5AC88149/5AC93322/5AC922E0" Ref="R21"  Part="1"
 AR Path="/5AC88149/5AC93462/5AC922E0" Ref="R26"  Part="1"
-F 0 "R21" V 5430 4500 50  0000 C CNN
+F 0 "R26" V 5430 4500 50  0000 C CNN
 F 1 "10k" V 5350 4500 50  0000 C CNN
 F 2 "Resistors_SMD:R_0603" V 5280 4500 50  0001 C CNN
@@
 $EndComp
 Wire Wire Line
-	3900 3800 3900 3700
+	3900 3700 3900 3800
 Wire Wire Line
 	5150 3750 3900 3750
@@
 Connection ~ 5050 3950
 $Comp
-L GND #PWR034
+L GND #PWR032
 U 1 1 5AC92519
 P 6000 3650
-AR Path="/5AC88149/5AC9150E/5AC92519" Ref="#PWR034"  Part="1"
-AR Path="/5AC88149/5AC931A3/5AC92519" Ref="#PWR041"  Part="1"
-AR Path="/5AC88149/5AC93322/5AC92519" Ref="#PWR048"  Part="1"
-AR Path="/5AC88149/5AC93462/5AC92519" Ref="#PWR055"  Part="1"
-F 0 "#PWR048" H 6000 3400 50  0001 C CNN
+AR Path="/5AC88149/5AC9150E/5AC92519" Ref="#PWR032"  Part="1"
+AR Path="/5AC88149/5AC931A3/5AC92519" Ref="#PWR039"  Part="1"
+AR Path="/5AC88149/5AC93322/5AC92519" Ref="#PWR046"  Part="1"
+AR Path="/5AC88149/5AC93462/5AC92519" Ref="#PWR053"  Part="1"
+F 0 "#PWR053" H 6000 3400 50  0001 C CNN
 F 1 "GND" H 6000 3500 50  0000 C CNN
 F 2 "" H 6000 3650 50  0001 C CNN
@@
 AR Path="/5AC88149/5AC93322/5AC9254A" Ref="R22"  Part="1"
 AR Path="/5AC88149/5AC93462/5AC9254A" Ref="R27"  Part="1"
-F 0 "R22" V 6280 3850 50  0000 C CNN
+F 0 "R27" V 6280 3850 50  0000 C CNN
 F 1 "2.4k" V 6200 3850 50  0000 C CNN
 F 2 "Resistors_SMD:R_0603" V 6130 3850 50  0001 C CNN
@@
 AR Path="/5AC88149/5AC93322/5AC925AA" Ref="R23"  Part="1"
 AR Path="/5AC88149/5AC93462/5AC925AA" Ref="R28"  Part="1"
-F 0 "R23" V 6780 4450 50  0000 C CNN
+F 0 "R28" V 6780 4450 50  0000 C CNN
 F 1 "5.1k" V 6700 4450 50  0000 C CNN
 F 2 "Resistors_SMD:R_0603" V 6630 4450 50  0001 C CNN
@@
 AR Path="/5AC88149/5AC93322/5AC9293D" Ref="C16"  Part="1"
 AR Path="/5AC88149/5AC93462/5AC9293D" Ref="C18"  Part="1"
-F 0 "C16" H 5125 3400 50  0000 L CNN
+F 0 "C18" H 5125 3400 50  0000 L CNN
 F 1 "100n" H 5125 3200 50  0000 L CNN
 F 2 "Capacitors_SMD:C_0603" H 5138 3150 50  0001 C CNN
@@
 AR Path="/5AC88149/5AC93322/5AC92986" Ref="C15"  Part="1"
 AR Path="/5AC88149/5AC93462/5AC92986" Ref="C17"  Part="1"
-F 0 "C15" H 4875 3400 50  0000 L CNN
+F 0 "C17" H 4875 3400 50  0000 L CNN
 F 1 "10u" H 4875 3200 50  0000 L CNN
 F 2 "Capacitors_SMD:C_0603" H 4888 3150 50  0001 C CNN
@@
 $EndComp
 $Comp
-L GND #PWR035
+L GND #PWR033
 U 1 1 5AC929C9
 P 4850 3450
-AR Path="/5AC88149/5AC9150E/5AC929C9" Ref="#PWR035"  Part="1"
-AR Path="/5AC88149/5AC931A3/5AC929C9" Ref="#PWR042"  Part="1"
-AR Path="/5AC88149/5AC93322/5AC929C9" Ref="#PWR049"  Part="1"
-AR Path="/5AC88149/5AC93462/5AC929C9" Ref="#PWR056"  Part="1"
-F 0 "#PWR049" H 4850 3200 50  0001 C CNN
+AR Path="/5AC88149/5AC9150E/5AC929C9" Ref="#PWR033"  Part="1"
+AR Path="/5AC88149/5AC931A3/5AC929C9" Ref="#PWR040"  Part="1"
+AR Path="/5AC88149/5AC93322/5AC929C9" Ref="#PWR047"  Part="1"
+AR Path="/5AC88149/5AC93462/5AC929C9" Ref="#PWR054"  Part="1"
+F 0 "#PWR054" H 4850 3200 50  0001 C CNN
 F 1 "GND" H 4850 3300 50  0000 C CNN
 F 2 "" H 4850 3450 50  0001 C CNN
@@
 Wire Wire Line
 	4850 3150 6650 3150
-Wire Wire Line
-	5350 3100 5350 3550
 Connection ~ 5100 3150
 Connection ~ 5350 3150
 Wire Wire Line
 	6650 3150 6650 3450
+Wire Wire Line
+	5350 3150 5350 3550
+$Comp
+L +5V #PWR041
+U 1 1 5ACAA528
+P 5350 3150
+AR Path="/5AC88149/5AC931A3/5ACAA528" Ref="#PWR041"  Part="1"
+AR Path="/5AC88149/5AC9150E/5ACAA528" Ref="#PWR034"  Part="1"
+AR Path="/5AC88149/5AC93322/5ACAA528" Ref="#PWR048"  Part="1"
+AR Path="/5AC88149/5AC93462/5ACAA528" Ref="#PWR055"  Part="1"
+F 0 "#PWR055" H 5350 3000 50  0001 C CNN
+F 1 "+5V" H 5350 3290 50  0000 C CNN
+F 2 "" H 5350 3150 50  0001 C CNN
+F 3 "" H 5350 3150 50  0001 C CNN
+	1    5350 3150
+	1    0    0    -1
+$EndComp
+$Comp
+L +5V #PWR042
+U 1 1 5ACAA596
+P 3900 3400
+AR Path="/5AC88149/5AC931A3/5ACAA596" Ref="#PWR042"  Part="1"
+AR Path="/5AC88149/5AC9150E/5ACAA596" Ref="#PWR035"  Part="1"
+AR Path="/5AC88149/5AC93322/5ACAA596" Ref="#PWR049"  Part="1"
+AR Path="/5AC88149/5AC93462/5ACAA596" Ref="#PWR056"  Part="1"
+F 0 "#PWR056" H 3900 3250 50  0001 C CNN
+F 1 "+5V" H 3900 3540 50  0000 C CNN
+F 2 "" H 3900 3400 50  0001 C CNN
+F 3 "" H 3900 3400 50  0001 C CNN
+	1    3900 3400
+	1    0    0    -1
+$EndComp
 $EndSCHEMATC

Commit message: Fixed transimpedance amps in schematic
Parts:
- added R32: 1.2k, Resistors_SMD:R_0603, symbol R
- R13: value 5.1k -> 2.4k
Connections:
- net GND: now also R12.2, R32.1; no longer U4.5 (+)
- net at R11.1, U4.1: now also U4.5 (+), R32.2; no longer R12.2
Other:
- moved on the sheet: C11, C12, R10, R11, R12, R13, R9, U4A, U4B

Commit message: Fixed transimpedance amp on layout and generated new Gerbers.
Parts:
- R11: value 10k -> 100k
Changed lines of the file:
@@
 LIBS:cmos4000
 LIBS:conn
+LIBS:logo
 LIBS:microchip_dspic33dsc
 LIBS:microchip_pic10mcu
@@
 LIBS:bosch
 LIBS:brooktre
+LIBS:Connector
 LIBS:contrib
 LIBS:cypress
@@
 LIBS:Diode
 LIBS:Display
+LIBS:driver_gate
 LIBS:dsp
+LIBS:DSP_Microchip_DSPIC33
 LIBS:elec-unifil
 LIBS:ESD_Protection
+LIBS:Espressif
+LIBS:FPGA_Actel
 LIBS:ftdi
 LIBS:gennum
+LIBS:Graphic
 LIBS:hc11
 LIBS:infineon
@@
 LIBS:ir
 LIBS:Lattice
+LIBS:LED
 LIBS:LEM
 LIBS:linear
+LIBS:Logic_74xgxx
+LIBS:Logic_74xx
+LIBS:Logic_CMOS_4000
+LIBS:Logic_CMOS_IEEE
 LIBS:logic_programmable
+LIBS:Logic_TTL_IEEE
 LIBS:maxim
+LIBS:MCU_Microchip_PIC10
+LIBS:MCU_Microchip_PIC12
+LIBS:MCU_Microchip_PIC16
+LIBS:MCU_Microchip_PIC18
+LIBS:MCU_Microchip_PIC24
+LIBS:MCU_Microchip_PIC32
+LIBS:MCU_NXP_Kinetis
+LIBS:MCU_NXP_LPC
+LIBS:MCU_NXP_S08
+LIBS:MCU_ST_STM8
+LIBS:MCU_ST_STM32
+LIBS:MCU_Texas_MSP430
 LIBS:Mechanical
 LIBS:memory
@@
 LIBS:microcontrollers
 LIBS:modules
+LIBS:Motor
 LIBS:motor_drivers
 LIBS:motorola
@@
 LIBS:references
 LIBS:regul
+LIBS:Relay
 LIBS:rfcom
 LIBS:RFSolutions
+LIBS:Sensor_Current
 LIBS:sensors
 LIBS:silabs
 LIBS:siliconi
 LIBS:supertex
+LIBS:Switch
 LIBS:texas
+LIBS:Transformer
+LIBS:Transistor
 LIBS:triac_thyristor
+LIBS:Valve
 LIBS:video
 LIBS:wiznet
@@
 $Descr A4 11693 8268
 encoding utf-8
-Sheet 6 6
+Sheet 5 6
 Title ""
 Date ""
@@
 AR Path="/5AC88149/5AC93322/5AC91533" Ref="U6"  Part="1"
 AR Path="/5AC88149/5AC93462/5AC91533" Ref="U7"  Part="1"
-F 0 "U4" H 4950 4050 50  0000 L CNN
+F 0 "U6" H 4950 4050 50  0000 L CNN
 F 1 "BA4510FVM-GTR" H 4950 3650 50  0000 L CNN
 F 2 "Housings_SSOP:MSOP-8_3x3mm_Pitch0.65mm" H 4950 3850 50  0001 C CNN
@@
 AR Path="/5AC88149/5AC93322/5AC9170A" Ref="U6"  Part="2"
 AR Path="/5AC88149/5AC93462/5AC9170A" Ref="U7"  Part="2"
-F 0 "U4" H 6750 4150 50  0000 L CNN
+F 0 "U6" H 6750 4150 50  0000 L CNN
 F 1 "BA4510FVM-GTR" H 6750 3750 50  0000 L CNN
 F 2 "Housings_SSOP:MSOP-8_3x3mm_Pitch0.65mm" H 6750 3950 50  0001 C CNN
@@
 AR Path="/5AC88149/5AC93322/5AC91801" Ref="#PWR043"  Part="1"
 AR Path="/5AC88149/5AC93462/5AC91801" Ref="#PWR050"  Part="1"
-F 0 "#PWR050" H 4850 3900 50  0001 C CNN
+F 0 "#PWR043" H 4850 3900 50  0001 C CNN
 F 1 "GND" H 4850 4000 50  0000 C CNN
 F 2 "" H 4850 4150 50  0001 C CNN
@@
 AR Path="/5AC88149/5AC93322/5AC91819" Ref="#PWR044"  Part="1"
 AR Path="/5AC88149/5AC93462/5AC91819" Ref="#PWR051"  Part="1"
-F 0 "#PWR051" H 6650 4000 50  0001 C CNN
+F 0 "#PWR044" H 6650 4000 50  0001 C CNN
 F 1 "GND" H 6650 4100 50  0000 C CNN
 F 2 "" H 6650 4250 50  0001 C CNN
@@
 AR Path="/5AC88149/5AC93322/5AC91C57" Ref="R20"  Part="1"
 AR Path="/5AC88149/5AC93462/5AC91C57" Ref="R25"  Part="1"
-F 0 "R10" V 3480 3950 50  0000 C CNN
+F 0 "R20" V 3480 3950 50  0000 C CNN
 F 1 "1M" V 3400 3950 50  0000 C CNN
 F 2 "Resistors_SMD:R_0603" V 3330 3950 50  0001 C CNN
@@
 AR Path="/5AC88149/5AC93322/5AC91CDA" Ref="R19"  Part="1"
 AR Path="/5AC88149/5AC93462/5AC91CDA" Ref="R24"  Part="1"
-F 0 "R9" V 3480 3550 50  0000 C CNN
+F 0 "R19" V 3480 3550 50  0000 C CNN
 F 1 "1M" V 3400 3550 50  0000 C CNN
 F 2 "Resistors_SMD:R_0603" V 3330 3550 50  0001 C CNN
@@
 AR Path="/5AC88149/5AC93322/5AC91D5F" Ref="#PWR045"  Part="1"
 AR Path="/5AC88149/5AC93462/5AC91D5F" Ref="#PWR052"  Part="1"
-F 0 "#PWR052" H 3400 3850 50  0001 C CNN
+F 0 "#PWR045" H 3400 3850 50  0001 C CNN
 F 1 "GND" H 3400 3950 50  0000 C CNN
 F 2 "" H 3400 4100 50  0001 C CNN
@@
 AR Path="/5AC88149/5AC93322/5AC922E0" Ref="R21"  Part="1"
 AR Path="/5AC88149/5AC93462/5AC922E0" Ref="R26"  Part="1"
-F 0 "R11" V 4930 4500 50  0000 C CNN
-F 1 "10k" V 4850 4500 50  0000 C CNN
+F 0 "R21" V 4930 4500 50  0000 C CNN
+F 1 "100k" V 4850 4500 50  0000 C CNN
 F 2 "Resistors_SMD:R_0603" V 4780 4500 50  0001 C CNN
 F 3 "" H 4850 4500 50  0001 C CNN
@@
 AR Path="/5AC88149/5AC93322/5AC9254A" Ref="R22"  Part="1"
 AR Path="/5AC88149/5AC93462/5AC9254A" Ref="R27"  Part="1"
-F 0 "R12" V 6280 4050 50  0000 C CNN
+F 0 "R22" V 6280 4050 50  0000 C CNN
 F 1 "2.4k" V 6200 4050 50  0000 C CNN
 F 2 "Resistors_SMD:R_0603" V 6130 4050 50  0001 C CNN
@@
 AR Path="/5AC88149/5AC93322/5AC925AA" Ref="R23"  Part="1"
 AR Path="/5AC88149/5AC93462/5AC925AA" Ref="R28"  Part="1"
-F 0 "R13" V 6780 4650 50  0000 C CNN
+F 0 "R23" V 6780 4650 50  0000 C CNN
 F 1 "2.4k" V 6700 4650 50  0000 C CNN
 F 2 "Resistors_SMD:R_0603" V 6630 4650 50  0001 C CNN
@@
 AR Path="/5AC88149/5AC93322/5AC9293D" Ref="C16"  Part="1"
 AR Path="/5AC88149/5AC93462/5AC9293D" Ref="C18"  Part="1"
-F 0 "C12" H 4625 3400 50  0000 L CNN
+F 0 "C16" H 4625 3400 50  0000 L CNN
 F 1 "100n" H 4625 3200 50  0000 L CNN
 F 2 "Capacitors_SMD:C_0603" H 4638 3150 50  0001 C CNN
@@
 AR Path="/5AC88149/5AC93322/5AC92986" Ref="C15"  Part="1"
 AR Path="/5AC88149/5AC93462/5AC92986" Ref="C17"  Part="1"
-F 0 "C11" H 4375 3400 50  0000 L CNN
+F 0 "C15" H 4375 3400 50  0000 L CNN
 F 1 "10u" H 4375 3200 50  0000 L CNN
 F 2 "Capacitors_SMD:C_0603" H 4388 3150 50  0001 C CNN
@@
 AR Path="/5AC88149/5AC93322/5AC929C9" Ref="#PWR046"  Part="1"
 AR Path="/5AC88149/5AC93462/5AC929C9" Ref="#PWR053"  Part="1"
-F 0 "#PWR053" H 4350 3200 50  0001 C CNN
+F 0 "#PWR046" H 4350 3200 50  0001 C CNN
 F 1 "GND" H 4350 3300 50  0000 C CNN
 F 2 "" H 4350 3450 50  0001 C CNN
@@
 AR Path="/5AC88149/5AC93322/5ACAA528" Ref="#PWR047"  Part="1"
 AR Path="/5AC88149/5AC93462/5ACAA528" Ref="#PWR054"  Part="1"
-F 0 "#PWR054" H 4850 3000 50  0001 C CNN
+F 0 "#PWR047" H 4850 3000 50  0001 C CNN
 F 1 "+5V" H 4850 3290 50  0000 C CNN
 F 2 "" H 4850 3150 50  0001 C CNN
@@
 AR Path="/5AC88149/5AC931A3/5ACE1471" Ref="#PWR041"  Part="1"
 AR Path="/5AC88149/5AC93322/5ACE1471" Ref="#PWR048"  Part="1"
-F 0 "#PWR055" H 6050 3800 50  0001 C CNN
+F 0 "#PWR048" H 6050 3800 50  0001 C CNN
 F 1 "GND" H 6050 3900 50  0000 C CNN
 F 2 "" H 6050 4050 50  0001 C CNN
@@
 AR Path="/5AC88149/5AC931A3/5ACE15E7" Ref="R30"  Part="1"
 AR Path="/5AC88149/5AC93322/5ACE15E7" Ref="R31"  Part="1"
-F 0 "R29" V 6480 3650 50  0000 C CNN
+F 0 "R31" V 6480 3650 50  0000 C CNN
 F 1 "1.2k" V 6400 3650 50  0000 C CNN
 F 2 "Resistors_SMD:R_0603" V 6330 3650 50  0001 C CNN
@@
 AR Path="/5AC88149/5AC931A3/5ACE1663" Ref="#PWR042"  Part="1"
 AR Path="/5AC88149/5AC93322/5ACE1663" Ref="#PWR049"  Part="1"
-F 0 "#PWR056" H 6250 3300 50  0001 C CNN
+F 0 "#PWR049" H 6250 3300 50  0001 C CNN
 F 1 "GND" H 6250 3400 50  0000 C CNN
 F 2 "" H 6250 3550 50  0001 C CNN
